File: pcb/circuit-design.kicad_pcb (KiCad board)
At the start: 2 copper layers, 9 parts, among them U1 ESP-01, U2 AMS1117-3.3

Commit message: Fixed something missing and improved a better visibility
Parts:
- C1: value 100uF -> 100uF 10v
- DHT: renamed from DHT11; value DHT11 -> DHT
Routing:
- net +3V3: track 71.3 -> 77.0 mm
Changed lines of the file:
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@@
     (property "Sheetname" "")
     (attr through_hole)
-    (fp_text reference "DHT11" (at -1.8455 -2.8055 -90) (layer "F.Cu")
-      (effects (font (size 1 1) (thickness 0.15)))
-    )
-    (fp_text value "DHT11" (at -0.3605 -4.2255 90) (layer "F.Fab") hide
+    (fp_text reference "DHT" (at 0.009 -1.41) (layer "F.Cu")
+      (effects (font (size 0.5 0.5) (thickness 0.125)))
+    )
+    (fp_text value "DHT" (at -0.3605 -4.2255 90) (layer "F.Fab") hide
       (effects (font (size 1 1) (thickness 0.15)))
     )
@@
       (effects (font (size 1 1) (thickness 0.15)))
     )
-    (fp_text value "AMS1117-3.3" (at -0.283 -5.5515) (layer "F.Cu")
-      (effects (font (size 1 1) (thickness 0.15) italic))
+    (fp_text value "AMS1117-3.3" (at 0.547 -4.0125) (layer "F.Cu")
+      (effects (font (size 0.5 0.5) (thickness 0.125) italic))
     )
     (fp_text user "${REFERENCE}" (at 0 0 90) (layer "F.Fab")
@@
     (property "Sheetname" "")
     (attr through_hole)
-    (fp_text reference "R1" (at 3.7645 0.0195) (layer "F.Cu")
-      (effects (font (size 1 1) (thickness 0.15)))
+    (fp_text reference "R1" (at 2.93 0) (layer "F.Cu")
+      (effects (font (size 0.6 0.95) (thickness 0.125)))
     )
     (fp_text value "4.7kOhm" (at 3.235 -3.775) (layer "F.Fab") hide
@@
     (property "Sheetname" "")
     (attr through_hole)
-    (fp_text reference "C1" (at -4.31 -0.035 180) (layer "F.Cu")
-      (effects (font (size 1 1) (thickness 0.15)))
-    )
-    (fp_text value "100uF" (at -5.89 0.055 180) (layer "F.Cu")
-      (effects (font (size 1 1) (thickness 0.15)))
+    (fp_text reference "C1" (at -2.58 -0.005 180) (layer "F.Cu")
+      (effects (font (size 0.5 0.5) (thickness 0.125)))
+    )
+    (fp_text value "100uF 10v" (at -3.739 0.105 180) (layer "F.Cu")
+      (effects (font (size 0.5 0.5) (thickness 0.125)))
     )
     (fp_text user "${REFERENCE}" (at -4 0.175 180) (layer "F.Fab") hide
@@
     )
     (fp_text value "ESP-01" (at 10.12 5.25 270) (layer "F.Cu")
-      (effects (font (size 1 1) (thickness 0.15)))
+      (effects (font (size 0.5 0.5) (thickness 0.15)))
     )
     (fp_line (start 1.27 -1.27) (end -1.27 -1.27) (layer "F.SilkS") (width 0.1524))
@@
     (fp_line (start -1.778 10.922) (end -1.778 -3.302) (layer "F.Fab") (width 0.05))
     (fp_line (start 22.86 -3.302) (end 22.86 10.922) (layer "F.Fab") (width 0.05))
-    (pad "1" thru_hole circle locked (at 0 0 90) (size 1.7272 1.7272) (drill 0.8) (layers *.Cu *.Mask)
+    (pad "1" thru_hole circle (at 0 0 90) (size 1.7272 1.7272) (drill 0.8) (layers *.Cu *.Mask)
       (net 6 "TX") (pinfunction "UTXD") (pintype "output"))
-    (pad "2" thru_hole rect locked (at 2.54 0 90) (size 1.7272 1.7272) (drill 1.016) (layers *.Cu *.Mask "F.SilkS")
+    (pad "2" thru_hole rect (at 2.54 0 90) (size 1.7272 1.7272) (drill 1.016) (layers *.Cu *.Mask "F.SilkS")
       (net 2 "GND") (pinfunction "GND") (pintype "power_in"))
-    (pad "3" thru_hole circle locked (at 0 2.54 90) (size 1.7272 1.7272) (drill 0.8) (layers *.Cu *.Mask)
+    (pad "3" thru_hole circle (at 0 2.54 90) (size 1.7272 1.7272) (drill 0.8) (layers *.Cu *.Mask)
       (net 3 "+3V3") (pinfunction "CH_PD") (pintype "input"))
-    (pad "4" thru_hole circle locked (at 2.54 2.54 90) (size 1.7272 1.7272) (drill 0.8) (layers *.Cu *.Mask)
+    (pad "4" thru_hole circle (at 2.54 2.54 90) (size 1.7272 1.7272) (drill 0.8) (layers *.Cu *.Mask)
       (net 5 "Net-(U1-Pad4)") (pinfunction "GPIO2") (pintype "tri_state"))
-    (pad "5" thru_hole oval locked (at 0 5.08 90) (size 0.5 0) (drill 0.8) (layers *.Cu *.Mask "F.SilkS")
+    (pad "5" thru_hole circle (at 0 5.08 90) (size 1 1) (drill 0.8) (layers *.Cu *.Mask)
       (net 7 "unconnected-(U1-Pad5)") (pinfunction "RST") (pintype "input"))
-    (pad "6" thru_hole circle locked (at 2.54 5.08 90) (size 1.7272 1.7272) (drill 0.8) (layers *.Cu *.Mask)
+    (pad "6" thru_hole circle (at 2.54 5.08 90) (size 1.7272 1.7272) (drill 0.8) (layers *.Cu *.Mask)
       (net 8 "RX") (pinfunction "GPIO0") (pintype "tri_state"))
-    (pad "7" thru_hole circle locked (at 0 7.62 90) (size 1.7272 1.7272) (drill 0.8) (layers *.Cu *.Mask)
+    (pad "7" thru_hole circle (at 0 7.62 90) (size 1.7272 1.7272) (drill 0.8) (layers *.Cu *.Mask)
       (net 3 "+3V3") (pinfunction "VCC") (pintype "power_in"))
-    (pad "8" thru_hole circle locked (at 2.54 7.62 90) (size 1.7272 1.7272) (drill 0.8) (layers *.Cu *.Mask)
+    (pad "8" thru_hole circle (at 2.54 7.62 90) (size 1.7272 1.7272) (drill 0.8) (layers *.Cu *.Mask)
       (net 9 "unconnected-(U1-Pad8)") (pinfunction "URXD") (pintype "input"))
   )
   (gr_rect (start 12.01 12.02) (end 62.15 62.11) (layer "User.1") (width 0.2) (fill none))
-  (gr_text "TX" (at 48.67 58.879) (layer "F.Cu")
-    (effects (font (size 1 1) (thickness 0.15)))
-  )
-  (gr_text "RX\n" (at 53.97 60.054) (layer "F.Cu")
-    (effects (font (size 1 1) (thickness 0.15)))
+  (gr_text "TX" (at 50.08 56.32) (layer "F.Cu")
+    (effects (font (size 0.4 0.4) (thickness 0.1)))
+  )
+  (gr_text "RX\n" (at 55.18 56.45) (layer "F.Cu")
+    (effects (font (size 0.4 0.4) (thickness 0.1)))
   )
   (segment (start 33.4825 21.593) (end 33.763 21.3125) (width 0.5) (layer "F.Cu") (net 1))
@@
   (segment (start 52.75 16.715) (end 52.75 19.351) (width 0.5) (layer "F.Cu") (net 3))
   (segment (start 51.28 57.414) (end 51.28 53.12) (width 0.5) (layer "F.Cu") (net 3))
+  (segment (start 43.435 14.7405) (end 40.063 18.1125) (width 0.5) (layer "F.Cu") (net 3))
   (segment (start 58.2736 51.37264) (end 58.15312 51.49312) (width 0.5) (layer "F.Cu") (net 3))
   (segment (start 52.75 19.351) (end 58.2736 24.8746) (width 0.5) (layer "F.Cu") (net 3))
@@
   (segment (start 27.325 18.941) (end 33.6915 18.941) (width 0.5) (layer "F.Cu") (net 3))
   (segment (start 58.07 51.41) (end 56.36 53.12) (width 0.5) (layer "F.Cu") (net 3))
+  (segment (start 40.063 18.1125) (end 40.063 19.0125) (width 0.5) (layer "F.Cu") (net 3))
   (segment (start 58.2736 24.8746) (end 58.2736 51.37264) (width 0.5) (layer "F.Cu") (net 3))
   (segment (start 50.21 22.71) (end 47.77 25.15) (width 0.5) (layer "F.Cu") (net 4))
@@
   (segment (start 53.82 50.58) (end 52.6314 51.7686) (width 0.5) (layer "F.Cu") (net 8))
   (zone (net 2) (net_name "GND") (layer "F.Cu") (hatch edge 0.508)
-    (connect_pads (clearance 0.8))
+    (connect_pads (clearance 0.75))
     (min_thickness 0.254) (filled_areas_thickness no)
-    (fill yes (thermal_gap 0.508) (thermal_bridge_width 0.508) (smoothing chamfer))
+    (fill yes (thermal_gap 0.508) (thermal_bridge_width 0.508))
     (polygon
       (pts
-        (xy 62.23 62.22)
-        (xy 11.93 62.16)
-        (xy 12.06 12.07)
-        (xy 62.13 12.07)
+        (xy 62.05 62.01)
+        (xy 12.11 62.01)
+        (xy 12.11 12.12)
+        (xy 62.05 12.12)
       )
     )
